Commit message: fixed the urdf issue with global frame, CoM and inertia

File: urdf/drone_v2.urdf (robot description, URDF)
Before this commit: robot drone_v2, 9 links, 7 joints
Joints:
- added joint joint_motor_front_right: type fixed, parent base_link, child link_motor_front_right, origin xyz=-0.053285 -0.13571 0.041658 rpy=1.5708 0 -2.979, axis 0 0 0
